File: straggio computer v1.3/NOTer and Rotate.sch (KiCad schematic (older format))
At the start: 0 parts

Commit message: Update 26/02/2021
Changed lines of the file:
@@
 $Descr A4 11693 8268
 encoding utf-8
-Sheet 33 53
+Sheet 50 53
 Title ""
 Date ""
@@
 Comment4 ""
 $EndDescr
+Text HLabel 1500 1000 0    50   Input ~ 0
+A_0
+Text HLabel 1500 1100 0    50   Input ~ 0
+A_1
+Text HLabel 1500 1200 0    50   Input ~ 0
+A_2
+Text HLabel 1500 1300 0    50   Input ~ 0
+A_3
+Text HLabel 1500 1400 0    50   Input ~ 0
+A_4
 Text HLabel 1500 1500 0    50   Input ~ 0
-In_0
+A_5
 Text HLabel 1500 1600 0    50   Input ~ 0
-In_1
+A_6
 Text HLabel 1500 1700 0    50   Input ~ 0
-In_2
+A_7
 Text HLabel 1500 1800 0    50   Input ~ 0
-In_3
+A_8
 Text HLabel 1500 1900 0    50   Input ~ 0
-In_4
+A_9
 Text HLabel 1500 2000 0    50   Input ~ 0
-In_5
+A_10
 Text HLabel 1500 2100 0    50   Input ~ 0
-In_6
+A_11
 Text HLabel 1500 2200 0    50   Input ~ 0
-In_7
+A_12
 Text HLabel 1500 2300 0    50   Input ~ 0
-In_8
+A_13
 Text HLabel 1500 2400 0    50   Input ~ 0
-In_9
+A_14
 Text HLabel 1500 2500 0    50   Input ~ 0
-In_10
-Text HLabel 1500 2600 0    50   Input ~ 0
-In_11
-Text HLabel 1500 2700 0    50   Input ~ 0
-In_12
+A_15
 Text HLabel 1500 2800 0    50   Input ~ 0
-In_13
+Enable_rotate_left
 Text HLabel 1500 2900 0    50   Input ~ 0
-In_14
+Enable_rotate_right
 Text HLabel 1500 3000 0    50   Input ~ 0
-In_15
+Enable_NOTer
+Text HLabel 1500 2650 0    50   Input ~ 0
+Rotate_carry_in
+Text HLabel 2000 1000 2    50   3State ~ 0
+C_0
+Text HLabel 2000 1100 2    50   3State ~ 0
+C_1
+Text HLabel 2000 1200 2    50   3State ~ 0
+C_2
+Text HLabel 2000 1300 2    50   3State ~ 0
+C_3
+Text HLabel 2000 1400 2    50   3State ~ 0
+C_4
 Text HLabel 2000 1500 2    50   3State ~ 0
-Out_0
+C_5
 Text HLabel 2000 1600 2    50   3State ~ 0
-Out_1
+C_6
 Text HLabel 2000 1700 2    50   3State ~ 0
-Out_2
+C_7
 Text HLabel 2000 1800 2    50   3State ~ 0
-Out_3
+C_8
 Text HLabel 2000 1900 2    50   3State ~ 0
-Out_4
+C_9
 Text HLabel 2000 2000 2    50   3State ~ 0
-Out_5
+C_10
 Text HLabel 2000 2100 2    50   3State ~ 0
-Out_6
+C_11
 Text HLabel 2000 2200 2    50   3State ~ 0
-Out_7
+C_12
 Text HLabel 2000 2300 2    50   3State ~ 0
-Out_8
+C_13
 Text HLabel 2000 2400 2    50   3State ~ 0
-Out_9
+C_14
 Text HLabel 2000 2500 2    50   3State ~ 0
-Out_10
-Text HLabel 2000 2600 2    50   3State ~ 0
-Out_11
-Text HLabel 2000 2700 2    50   3State ~ 0
-Out_12
-Text HLabel 2000 2800 2    50   3State ~ 0
-Out_13
-Text HLabel 2000 2900 2    50   3State ~ 0
-Out_14
-Text HLabel 2000 3000 2    50   3State ~ 0
-Out_15
+C_15
+Text HLabel 2000 2650 2    50   3State ~ 0
+Rotate_carry_out
 $EndSCHEMATC
