File: straggio computer v1.3/Multiplier.sch (KiCad schematic (older format))
At the start: 0 parts

Commit message: update
Changed lines of the file:
@@
 $Descr A4 11693 8268
 encoding utf-8
-Sheet 49 60
+Sheet 46 60
 Title ""
 Date ""
@@
 Text HLabel 1500 3050 0    50   Input ~ 0
 B_4
+Text HLabel 1500 3250 0    50   Input ~ 0
+B_6
 Text HLabel 1500 3150 0    50   Input ~ 0
 B_5
-Text HLabel 1500 3250 0    50   Input ~ 0
-B_6
 Text HLabel 1500 3350 0    50   Input ~ 0
 B_7
@@
 Text HLabel 1500 4150 0    50   Input ~ 0
 B_15
-Text HLabel 1500 4350 0    50   Input ~ 0
-Bus_A_pull_down
-Text HLabel 1500 4450 0    50   Input ~ 0
-Zero_carry_in
-Text HLabel 1500 4550 0    50   Input ~ 0
-adder_carry_in
-Text HLabel 1500 4650 0    50   Input ~ 0
-Enable_adder
-Text HLabel 2500 1000 2    50   3State ~ 0
+Text HLabel 2500 1000 2    50   Output ~ 0
 C_0
-Text HLabel 2500 1100 2    50   3State ~ 0
+Text HLabel 2500 1100 2    50   Output ~ 0
 C_1
-Text HLabel 2500 1200 2    50   3State ~ 0
+Text HLabel 2500 1200 2    50   Output ~ 0
 C_2
-Text HLabel 2500 1300 2    50   3State ~ 0
+Text HLabel 2500 1300 2    50   Output ~ 0
 C_3
-Text HLabel 2500 1400 2    50   3State ~ 0
+Text HLabel 2500 1400 2    50   Output ~ 0
 C_4
-Text HLabel 2500 1500 2    50   3State ~ 0
+Text HLabel 2500 1500 2    50   Output ~ 0
 C_5
-Text HLabel 2500 1600 2    50   3State ~ 0
+Text HLabel 2500 1600 2    50   Output ~ 0
 C_6
-Text HLabel 2500 1700 2    50   3State ~ 0
+Text HLabel 2500 1700 2    50   Output ~ 0
 C_7
-Text HLabel 2500 1800 2    50   3State ~ 0
+Text HLabel 2500 1800 2    50   Output ~ 0
 C_8
-Text HLabel 2500 1900 2    50   3State ~ 0
+Text HLabel 2500 1900 2    50   Output ~ 0
 C_9
-Text HLabel 2500 2000 2    50   3State ~ 0
+Text HLabel 2500 2000 2    50   Output ~ 0
 C_10
-Text HLabel 2500 2100 2    50   3State ~ 0
+Text HLabel 2500 2100 2    50   Output ~ 0
 C_11
-Text HLabel 2500 2200 2    50   3State ~ 0
+Text HLabel 2500 2200 2    50   Output ~ 0
 C_12
-Text HLabel 2500 2300 2    50   3State ~ 0
+Text HLabel 2500 2300 2    50   Output ~ 0
 C_13
-Text HLabel 2500 2400 2    50   3State ~ 0
+Text HLabel 2500 2400 2    50   Output ~ 0
 C_14
-Text HLabel 2500 2500 2    50   3State ~ 0
+Text HLabel 2500 2500 2    50   Output ~ 0
 C_15
-Text HLabel 2500 2650 2    50   Output ~ 0
-adder_carry_out
+Text HLabel 2500 2600 2    50   Output ~ 0
+C_16
+Text HLabel 2500 2700 2    50   Output ~ 0
+C_17
+Text HLabel 2500 2800 2    50   Output ~ 0
+C_18
+Text HLabel 2500 2900 2    50   Output ~ 0
+C_19
+Text HLabel 2500 3000 2    50   Output ~ 0
+C_20
+Text HLabel 2500 3100 2    50   Output ~ 0
+C_21
+Text HLabel 2500 3200 2    50   Output ~ 0
+C_22
+Text HLabel 2500 3300 2    50   Output ~ 0
+C_23
+Text HLabel 2500 3400 2    50   Output ~ 0
+C_24
+Text HLabel 2500 3500 2    50   Output ~ 0
+C_25
+Text HLabel 2500 3600 2    50   Output ~ 0
+C_26
+Text HLabel 2500 3700 2    50   Output ~ 0
+C_27
+Text HLabel 2500 3800 2    50   Output ~ 0
+C_28
+Text HLabel 2500 3900 2    50   Output ~ 0
+C_29
+Text HLabel 2500 4000 2    50   Output ~ 0
+C_30
+Text HLabel 2500 4100 2    50   Output ~ 0
+C_31
+Text HLabel 1500 4300 0    50   Input ~ 0
+Enable_multiplier
 $EndSCHEMATC
