File: straggio computer v1.3/NOTer Rotate and Shift.sch (KiCad schematic (older format))
At the start: 0 parts

Commit message: update
Changed lines of the file:
@@
 Text HLabel 1500 2900 0    50   Input ~ 0
 Enable_rotate_right
-Text HLabel 1500 3000 0    50   Input ~ 0
+Text HLabel 1500 3550 0    50   Input ~ 0
 Enable_NOTer
 Text HLabel 1500 2650 0    50   Input ~ 0
@@
 Text HLabel 2000 2650 2    50   3State ~ 0
 Rotate_carry_out
+Text HLabel 1500 3100 0    50   Input ~ 0
+Enable_shift_left_with_0
+Text HLabel 1500 3200 0    50   Input ~ 0
+Enable_shift_right_with_0
+Text HLabel 1500 3300 0    50   Input ~ 0
+Enable_shift_left_with_1
+Text HLabel 1500 3400 0    50   Input ~ 0
+Enable_shift_right_with_1
 $EndSCHEMATC

Commit message: update
Parts:
- added C? (x2): C, symbol Device:C
- added J?: Input A, symbol Connector:Conn_01x16_Male
- added J?: Output C, symbol Connector:Conn_01x16_Male
- added J?: Control signals, symbol Connector:Conn_01x08_Male
- added J?: Control signal, symbol Connector:Conn_01x01_Male
- added J?: Power, symbol Connector:Conn_01x02_Male
- added Q? (x235): 2N7000, Package_TO_SOT_THT:TO-92_Inline, symbol Transistor_FET:2N7000
- added R? (x177): R, symbol Device:R
Connections:
- net A_0: now also J?.1 (Pin_1), Q?.2 (G), Q?.2 (G), Q?.2 (G)
- net A_1: now also J?.2 (Pin_2), Q?.2 (G), Q?.2 (G), Q?.2 (G)
- net A_10: now also J?.11 (Pin_11), Q?.2 (G), Q?.2 (G), Q?.2 (G)
- net A_11: now also J?.12 (Pin_12), Q?.2 (G), Q?.2 (G), Q?.2 (G)
- net A_12: now also J?.13 (Pin_13), Q?.2 (G), Q?.2 (G), Q?.2 (G)
- net A_13: now also J?.14 (Pin_14), Q?.2 (G), Q?.2 (G), Q?.2 (G)
- net A_14: now also J?.15 (Pin_15), Q?.2 (G), Q?.2 (G), Q?.2 (G)
- net A_15: now also J?.16 (Pin_16), Q?.2 (G), Q?.2 (G), Q?.2 (G)
- net A_2: now also J?.3 (Pin_3), Q?.2 (G), Q?.2 (G), Q?.2 (G)
- net A_3: now also J?.4 (Pin_4), Q?.2 (G), Q?.2 (G), Q?.2 (G)
- net A_4: now also J?.5 (Pin_5), Q?.2 (G), Q?.2 (G), Q?.2 (G)
- net A_5: now also J?.6 (Pin_6), Q?.2 (G), Q?.2 (G), Q?.2 (G)
- net A_6: now also J?.7 (Pin_7), Q?.2 (G), Q?.2 (G), Q?.2 (G)
- net A_7: now also J?.8 (Pin_8), Q?.2 (G), Q?.2 (G), Q?.2 (G)
- net A_8: now also J?.9 (Pin_9), Q?.2 (G), Q?.2 (G), Q?.2 (G)
- net A_9: now also J?.10 (Pin_10), Q?.2 (G), Q?.2 (G), Q?.2 (G)
- net C_0: now also J?.16 (Pin_16), Q?.3 (D), Q?.3 (D), Q?.3 (D), R?.2, R?.2, R?.2
- net C_1: now also J?.15 (Pin_15), Q?.3 (D), Q?.3 (D), Q?.3 (D), R?.2, R?.2, R?.2
- net C_10: now also J?.6 (Pin_6), Q?.3 (D), Q?.3 (D), Q?.3 (D), R?.2, R?.2, R?.2
- net C_11: now also J?.5 (Pin_5), Q?.3 (D), Q?.3 (D), Q?.3 (D), R?.2, R?.2, R?.2
- net C_12: now also J?.4 (Pin_4), Q?.3 (D), Q?.3 (D), Q?.3 (D), R?.2, R?.2, R?.2
- net C_13: now also J?.3 (Pin_3), Q?.3 (D), Q?.3 (D), Q?.3 (D), R?.2, R?.2, R?.2
- net C_14: now also J?.2 (Pin_2), Q?.3 (D), Q?.3 (D), Q?.3 (D), R?.2, R?.2, R?.2
- net C_15: now also J?.1 (Pin_1), Q?.3 (D), Q?.3 (D), Q?.3 (D), R?.2, R?.2, R?.2
- net C_2: now also J?.14 (Pin_14), Q?.3 (D), Q?.3 (D), Q?.3 (D), R?.2, R?.2, R?.2
- net C_3: now also J?.13 (Pin_13), Q?.3 (D), Q?.3 (D), Q?.3 (D), R?.2, R?.2, R?.2
- net C_4: now also J?.12 (Pin_12), Q?.3 (D), Q?.3 (D), Q?.3 (D), R?.2, R?.2, R?.2
- net C_5: now also J?.11 (Pin_11), Q?.3 (D), Q?.3 (D), Q?.3 (D), R?.2, R?.2, R?.2
- net C_6: now also J?.10 (Pin_10), Q?.3 (D), Q?.3 (D), Q?.3 (D), R?.2, R?.2, R?.2
- net C_7: now also J?.9 (Pin_9), Q?.3 (D), Q?.3 (D), Q?.3 (D), R?.2, R?.2, R?.2
- net C_8: now also J?.8 (Pin_8), Q?.3 (D), Q?.3 (D), Q?.3 (D), R?.2, R?.2, R?.2
- net C_9: now also J?.7 (Pin_7), Q?.3 (D), Q?.3 (D), Q?.3 (D), R?.2, R?.2, R?.2
- net Enable_NOTer: now also J?.8 (Pin_8), Q?.2 (G), Q?.2 (G), Q?.2 (G), Q?.2 (G), Q?.2 (G), Q?.2 (G), Q?.2 (G), Q?.2 (G), Q?.2 (G), Q?.2 (G), Q?.2 (G), Q?.2 (G), Q?.2 (G), Q?.2 (G), Q?.2 (G), Q?.2 (G)
- net Enable_rotate_left: now also J?.7 (Pin_7), Q?.2 (G)
- net Enable_rotate_right: now also J?.4 (Pin_4), Q?.2 (G)
- net Enable_shift_left_with_0: now also J?.5 (Pin_5), Q?.2 (G), Q?.2 (G)
- net Enable_shift_left_with_1: now also J?.6 (Pin_6), Q?.2 (G), Q?.2 (G)
- net Enable_shift_right_with_0: now also J?.2 (Pin_2), Q?.2 (G), Q?.2 (G)
- net Enable_shift_right_with_1: now also J?.3 (Pin_3), Q?.2 (G), Q?.2 (G)
- net Rotate_carry_in: now also J?.1 (Pin_1), Q?.2 (G)
- net Rotate_carry_out: now also J?.1 (Pin_1), Q?.3 (D), Q?.3 (D), R?.2, R?.2
- new net: Q?.2 (G), Q?.3 (D), Q?.3 (D), R?.2 (x51)
- new net: Q?.2 (G), Q?.3 (D), R?.2 (x70)
- new net: Q?.2 (G), Q?.2 (G), Q?.2 (G), Q?.2 (G), Q?.2 (G), Q?.2 (G), Q?.2 (G), Q?.2 (G), Q?.2 (G), Q?.2 (G), Q?.2 (G), Q?.2 (G), Q?.2 (G), Q?.2 (G), Q?.2 (G), Q?.2 (G), Q?.2 (G), Q?.3 (D), R?.2 (x2)
- new net: Q?.2 (G), Q?.2 (G), Q?.3 (D), R?.2
- new net: Q?.1 (S), Q?.3 (D)
- new net: Q?.2 (G), Q?.3 (D), Q?.3 (D), Q?.3 (D), R?.2 (x3)
- new net GND: C?.2, C?.2, J?.2 (Pin_2), Q?.1 (S), Q?.1 (S), Q?.1 (S), Q?.1 (S), Q?.1 (S), Q?.1 (S), Q?.1 (S), Q?.1 (S), Q?.1 (S), Q?.1 (S), Q?.1 (S), Q?.1 (S), Q?.1 (S), Q?.1 (S), Q?.1 (S), Q?.1 (S), Q?.1 (S), Q?.1 (S), Q?.1 (S), Q?.1 (S), Q?.1 (S), Q?.1 (S), Q?.1 (S), Q?.1 (S), Q?.1 (S), Q?.1 (S), Q?.1 (S), Q?.1 (S), Q?.1 (S), Q?.1 (S), Q?.1 (S), Q?.1 (S), Q?.1 (S), Q?.1 (S), Q?.1 (S), Q?.1 (S), Q?.1 (S), Q?.1 (S), Q?.1 (S), Q?.1 (S), Q?.1 (S), Q?.1 (S), Q?.1 (S), Q?.1 (S), Q?.1 (S), Q?.1 (S), Q?.1 (S), Q?.1 (S), Q?.1 (S), Q?.1 (S), Q?.1 (S), Q?.1 (S), Q?.1 (S), Q?.1 (S), Q?.1 (S), Q?.1 (S), Q?.1 (S), Q?.1 (S), Q?.1 (S), Q?.1 (S), Q?.1 (S), Q?.1 (S), Q?.1 (S), Q?.1 (S), Q?.1 (S), Q?.1 (S), Q?.1 (S), Q?.1 (S), Q?.1 (S), Q?.1 (S), Q?.1 (S), Q?.1 (S), Q?.1 (S), Q?.1 (S), Q?.1 (S), Q?.1 (S), Q?.1 (S), Q?.1 (S), Q?.1 (S), Q?.1 (S), Q?.1 (S), Q?.1 (S), Q?.1 (S), Q?.1 (S), Q?.1 (S), Q?.1 (S), Q?.1 (S), Q?.1 (S), Q?.1 (S), Q?.1 (S), Q?.1 (S), Q?.1 (S), Q?.1 (S), Q?.1 (S), Q?.1 (S), Q?.1 (S), Q?.1 (S), Q?.1 (S), Q?.1 (S), Q?.1 (S), Q?.1 (S), Q?.1 (S), Q?.1 (S), Q?.1 (S), Q?.1 (S), Q?.1 (S), Q?.1 (S), Q?.1 (S), Q?.1 (S), Q?.1 (S), Q?.1 (S), Q?.1 (S), Q?.1 (S), Q?.1 (S), Q?.1 (S), Q?.1 (S), Q?.1 (S), Q?.1 (S), Q?.1 (S), Q?.1 (S), Q?.1 (S), Q?.1 (S), Q?.1 (S), Q?.1 (S), Q?.1 (S), Q?.1 (S), Q?.1 (S), Q?.1 (S), Q?.1 (S), Q?.1 (S), Q?.1 (S), Q?.1 (S), Q?.1 (S), Q?.1 (S), Q?.1 (S), Q?.1 (S), Q?.1 (S), Q?.1 (S), Q?.1 (S), Q?.1 (S), Q?.1 (S), Q?.1 (S), Q?.1 (S), Q?.1 (S), Q?.1 (S), Q?.1 (S), Q?.1 (S), Q?.1 (S), Q?.1 (S), Q?.1 (S), Q?.1 (S), Q?.1 (S), Q?.1 (S), Q?.1 (S), Q?.1 (S), Q?.1 (S), Q?.1 (S), Q?.1 (S), Q?.1 (S), Q?.1 (S), Q?.1 (S), Q?.1 (S), Q?.1 (S), Q?.1 (S), Q?.1 (S), Q?.1 (S), Q?.1 (S), Q?.1 (S), Q?.1 (S), Q?.1 (S), Q?.1 (S), Q?.1 (S), Q?.1 (S), Q?.1 (S), Q?.1 (S), Q?.1 (S), Q?.1 (S), Q?.1 (S), Q?.1 (S), Q?.1 (S), Q?.1 (S), Q?.1 (S), Q?.1 (S), Q?.1 (S), Q?.1 (S), Q?.1 (S), Q?.1 (S), Q?.1 (S), Q?.1 (S), Q?.1 (S), Q?.1 (S), Q?.1 (S), Q?.1 (S), Q?.1 (S), Q?.1 (S), Q?.1 (S), Q?.1 (S), Q?.1 (S), Q?.1 (S), Q?.1 (S), Q?.1 (S), Q?.1 (S), Q?.1 (S), Q?.1 (S), Q?.1 (S), Q?.1 (S), Q?.1 (S), Q?.1 (S), Q?.1 (S), Q?.1 (S), Q?.1 (S), Q?.1 (S), Q?.1 (S), Q?.1 (S), Q?.1 (S), Q?.1 (S), Q?.1 (S), Q?.1 (S), Q?.1 (S), Q?.1 (S), Q?.1 (S), Q?.1 (S), Q?.1 (S), Q?.1 (S), Q?.1 (S), Q?.1 (S), Q?.1 (S), Q?.1 (S), Q?.1 (S), Q?.1 (S), Q?.1 (S), Q?.1 (S), Q?.1 (S), Q?.1 (S)
- new net VDD: C?.1, C?.1, J?.1 (Pin_1), R?.1, R?.1, R?.1, R?.1, R?.1, R?.1, R?.1, R?.1, R?.1, R?.1, R?.1, R?.1, R?.1, R?.1, R?.1, R?.1, R?.1, R?.1, R?.1, R?.1, R?.1, R?.1, R?.1, R?.1, R?.1, R?.1, R?.1, R?.1, R?.1, R?.1, R?.1, R?.1, R?.1, R?.1, R?.1, R?.1, R?.1, R?.1, R?.1, R?.1, R?.1, R?.1, R?.1, R?.1, R?.1, R?.1, R?.1, R?.1, R?.1, R?.1, R?.1, R?.1, R?.1, R?.1, R?.1, R?.1, R?.1, R?.1, R?.1, R?.1, R?.1, R?.1, R?.1, R?.1, R?.1, R?.1, R?.1, R?.1, R?.1, R?.1, R?.1, R?.1, R?.1, R?.1, R?.1, R?.1, R?.1, R?.1, R?.1, R?.1, R?.1, R?.1, R?.1, R?.1, R?.1, R?.1, R?.1, R?.1, R?.1, R?.1, R?.1, R?.1, R?.1, R?.1, R?.1, R?.1, R?.1, R?.1, R?.1, R?.1, R?.1, R?.1, R?.1, R?.1, R?.1, R?.1, R?.1, R?.1, R?.1, R?.1, R?.1, R?.1, R?.1, R?.1, R?.1, R?.1, R?.1, R?.1, R?.1, R?.1, R?.1, R?.1, R?.1, R?.1, R?.1, R?.1, R?.1, R?.1, R?.1, R?.1, R?.1, R?.1, R?.1, R?.1, R?.1, R?.1, R?.1, R?.1, R?.1, R?.1, R?.1, R?.1, R?.1, R?.1, R?.1, R?.1, R?.1, R?.1, R?.1, R?.1, R?.1, R?.1, R?.1, R?.1, R?.1, R?.1, R?.1, R?.1, R?.1, R?.1, R?.1, R?.1, R?.1, R?.1, R?.1, R?.1, R?.1, R?.1, R?.1, R?.1, R?.1, R?.1, R?.1, R?.1, R?.1, R?.1, R?.1
Other:
- note added: "3 input OR"
- note added: "AND"
- note added: "Cy"
- note added: "En_l"
- note added: "En_r"
- note added: "Enabler"
- note added: "Left operation"
- note added: "NOT"
- note added: "NOTer"
- note added: "OR"
- note added: "Rotate/Shift left"
- note added: "Rotate/Shift right"
- note added: "right operation"
