File: straggio computer v1.3/full 8bit register.sch (KiCad schematic (older format))
At the start: 0 parts

Commit message: Update 22/02/2021
Parts:
- added C? (x2): C, symbol Device:C
- added J?: control, symbol Connector:Conn_01x02_Male
- added J?: Input, symbol Connector:Conn_01x08_Male
- added J?: Output, symbol Connector:Conn_01x08_Male
- added J?: power, symbol Connector:Conn_01x02_Male
- added Q? (x96): 2N7000, Package_TO_SOT_THT:TO-92_Inline, symbol Transistor_FET:2N7000
- added R? (x56): R, symbol Device:R
Connections:
- net Enable_register: now also J?.1 (Pin_1), Q?.2 (G), Q?.2 (G), Q?.2 (G), Q?.2 (G), Q?.2 (G), Q?.2 (G), Q?.2 (G), Q?.2 (G)
- net In_0: now also J?.1 (Pin_1), Q?.2 (G)
- net In_1: now also J?.2 (Pin_2), Q?.2 (G)
- net In_2: now also J?.3 (Pin_3), Q?.2 (G)
- net In_3: now also J?.4 (Pin_4), Q?.2 (G)
- net In_4: now also J?.5 (Pin_5), Q?.2 (G)
- net In_5: now also J?.6 (Pin_6), Q?.2 (G)
- net In_6: now also J?.7 (Pin_7), Q?.2 (G)
- net In_7: now also J?.8 (Pin_8), Q?.2 (G)
- net Out_0: now also J?.8 (Pin_8), Q?.3 (D), R?.2
- net Out_1: now also J?.7 (Pin_7), Q?.3 (D), R?.2
- net Out_2: now also J?.6 (Pin_6), Q?.3 (D), R?.2
- net Out_3: now also J?.5 (Pin_5), Q?.3 (D), R?.2
- net Out_4: now also J?.4 (Pin_4), Q?.3 (D), R?.2
- net Out_5: now also J?.3 (Pin_3), Q?.3 (D), R?.2
- net Out_6: now also J?.2 (Pin_2), Q?.3 (D), R?.2
- net Out_7: now also J?.1 (Pin_1), Q?.3 (D), R?.2
- net Set_register: now also J?.2 (Pin_2), Q?.2 (G), Q?.2 (G), Q?.2 (G), Q?.2 (G), Q?.2 (G), Q?.2 (G), Q?.2 (G), Q?.2 (G), Q?.2 (G), Q?.2 (G), Q?.2 (G), Q?.2 (G), Q?.2 (G), Q?.2 (G), Q?.2 (G), Q?.2 (G)
- new net: Q?.1 (S), Q?.3 (D) (x32)
- new net: Q?.2 (G), Q?.2 (G), Q?.3 (D), R?.2 (x16)
- new net: Q?.2 (G), Q?.3 (D), R?.2 (x24)
- new net: Q?.2 (G), Q?.3 (D), Q?.3 (D), R?.2 (x8)
- new net GND: C?.2, C?.2, J?.2 (Pin_2), Q?.1 (S), Q?.1 (S), Q?.1 (S), Q?.1 (S), Q?.1 (S), Q?.1 (S), Q?.1 (S), Q?.1 (S), Q?.1 (S), Q?.1 (S), Q?.1 (S), Q?.1 (S), Q?.1 (S), Q?.1 (S), Q?.1 (S), Q?.1 (S), Q?.1 (S), Q?.1 (S), Q?.1 (S), Q?.1 (S), Q?.1 (S), Q?.1 (S), Q?.1 (S), Q?.1 (S), Q?.1 (S), Q?.1 (S), Q?.1 (S), Q?.1 (S), Q?.1 (S), Q?.1 (S), Q?.1 (S), Q?.1 (S), Q?.1 (S), Q?.1 (S), Q?.1 (S), Q?.1 (S), Q?.1 (S), Q?.1 (S), Q?.1 (S), Q?.1 (S), Q?.1 (S), Q?.1 (S), Q?.1 (S), Q?.1 (S), Q?.1 (S), Q?.1 (S), Q?.1 (S), Q?.1 (S), Q?.1 (S), Q?.1 (S), Q?.1 (S), Q?.1 (S), Q?.1 (S), Q?.1 (S), Q?.1 (S), Q?.1 (S), Q?.1 (S), Q?.1 (S), Q?.1 (S), Q?.1 (S), Q?.1 (S), Q?.1 (S), Q?.1 (S), Q?.1 (S)
- new net VDD: C?.1, C?.1, J?.1 (Pin_1), R?.1, R?.1, R?.1, R?.1, R?.1, R?.1, R?.1, R?.1, R?.1, R?.1, R?.1, R?.1, R?.1, R?.1, R?.1, R?.1, R?.1, R?.1, R?.1, R?.1, R?.1, R?.1, R?.1, R?.1, R?.1, R?.1, R?.1, R?.1, R?.1, R?.1, R?.1, R?.1, R?.1, R?.1, R?.1, R?.1, R?.1, R?.1, R?.1, R?.1, R?.1, R?.1, R?.1, R?.1, R?.1, R?.1, R?.1, R?.1, R?.1, R?.1, R?.1, R?.1, R?.1, R?.1, R?.1, R?.1
Other:
- note added: "ENABLER"
- note added: "MEMORY CELL"
