File: straggio computer v1.3/straggio computer v1.3.sch (KiCad schematic (older format))
At the start: 0 parts

Commit message: Update 22/02/2021
Other:
- note added: "sch ="
Changed lines of the file:
@@
 $Descr A2 23386 16535
 encoding utf-8
-Sheet 1 35
+Sheet 1 39
 Title ""
 Date ""
@@
 $EndDescr
 $Sheet
-S 10950 9800 1100 5000
+S 11000 8000 1100 5000
 U 603298DA
 F0 "work registers" 50
 F1 "work registers.sch" 50
-F2 "In_bus_0" I L 10950 9900 50
-F3 "In_bus_1" I L 10950 10000 50
-F4 "In_bus_2" I L 10950 10100 50
-F5 "In_bus_3" I L 10950 10200 50
-F6 "In_bus_4" I L 10950 10300 50
-F7 "In_bus_5" I L 10950 10400 50
-F8 "In_bus_6" I L 10950 10500 50
-F9 "In_bus_7" I L 10950 10600 50
-F10 "In_bus_8" I L 10950 10700 50
-F11 "In_bus_9" I L 10950 10800 50
-F12 "In_bus_10" I L 10950 10900 50
-F13 "In_bus_11" I L 10950 11000 50
-F14 "In_bus_12" I L 10950 11100 50
-F15 "In_bus_13" I L 10950 11200 50
-F16 "In_bus_14" I L 10950 11300 50
-F17 "In_bus_15" I L 10950 11400 50
-F18 "Set_reg_R0" I L 10950 11550 50
-F19 "Set_reg_R1" I L 10950 11650 50
-F20 "Set_reg_R2" I L 10950 11750 50
-F21 "Set_reg_R3" I L 10950 11850 50
-F22 "Set_reg_R4" I L 10950 11950 50
-F23 "Set_reg_R5" I L 10950 12050 50
-F24 "Set_reg_R6" I L 10950 12150 50
-F25 "Set_reg_R7" I L 10950 12250 50
-F26 "Set_reg_R8" I L 10950 12350 50
-F27 "Set_reg_R9" I L 10950 12450 50
-F28 "Set_reg_R10" I L 10950 12550 50
-F29 "Set_reg_R11" I L 10950 12650 50
-F30 "Set_reg_R12" I L 10950 12750 50
-F31 "Set_reg_R13" I L 10950 12850 50
-F32 "Set_reg_R14" I L 10950 12950 50
-F33 "Set_reg_R15" I L 10950 13050 50
-F34 "Enbale_reg_R0" I L 10950 13200 50
-F35 "Enable_reg_R1" I L 10950 13300 50
-F36 "Enable_reg_R2" I L 10950 13400 50
-F37 "Enable_reg_R3" I L 10950 13500 50
-F38 "Enable_reg_R4" I L 10950 13600 50
-F39 "Enable_reg_R5" I L 10950 13700 50
-F40 "Enable_reg_R6" I L 10950 13800 50
-F41 "Enable_reg_R7" I L 10950 13900 50
-F42 "Enable_reg_R8" I L 10950 14000 50
-F43 "Enable_reg_R9" I L 10950 14100 50
-F44 "Enable_reg_R10" I L 10950 14200 50
-F45 "Enable_reg_R11" I L 10950 14300 50
-F46 "Enable_reg_R12" I L 10950 14400 50
-F47 "Enable_reg_R13" I L 10950 14500 50
-F48 "Enable_reg_R14" I L 10950 14600 50
-F49 "Enable_reg_R15" I L 10950 14700 50
-F50 "Out_bus_0" T R 12050 9900 50
-F51 "Out_bus_1" T R 12050 10000 50
-F52 "Out_bus_2" T R 12050 10100 50
-F53 "Out_bus_3" T R 12050 10200 50
-F54 "Out_bus_4" T R 12050 10300 50
-F55 "Out_bus_5" T R 12050 10400 50
-F56 "Out_bus_6" T R 12050 10500 50
-F57 "Out_bus_7" T R 12050 10600 50
-F58 "Out_bus_8" T R 12050 10700 50
-F59 "Out_bus_9" T R 12050 10800 50
-F60 "Out_bus_10" T R 12050 10900 50
-F61 "Out_bus_11" T R 12050 11000 50
-F62 "Out_bus_12" T R 12050 11100 50
-F63 "Out_bus_13" T R 12050 11200 50
-F64 "Out_bus_14" T R 12050 11300 50
-F65 "Out_bus_15" T R 12050 11400 50
+F2 "In_bus_0" I L 11000 8100 50
+F3 "In_bus_1" I L 11000 8200 50
+F4 "In_bus_2" I L 11000 8300 50
+F5 "In_bus_3" I L 11000 8400 50
+F6 "In_bus_4" I L 11000 8500 50
+F7 "In_bus_5" I L 11000 8600 50
+F8 "In_bus_6" I L 11000 8700 50
+F9 "In_bus_7" I L 11000 8800 50
+F10 "In_bus_8" I L 11000 8900 50
+F11 "In_bus_9" I L 11000 9000 50
+F12 "In_bus_10" I L 11000 9100 50
+F13 "In_bus_11" I L 11000 9200 50
+F14 "In_bus_12" I L 11000 9300 50
+F15 "In_bus_13" I L 11000 9400 50
+F16 "In_bus_14" I L 11000 9500 50
+F17 "In_bus_15" I L 11000 9600 50
+F18 "Set_reg_R0" I L 11000 9750 50
+F19 "Set_reg_R1" I L 11000 9850 50
+F20 "Set_reg_R2" I L 11000 9950 50
+F21 "Set_reg_R3" I L 11000 10050 50
+F22 "Set_reg_R4" I L 11000 10150 50
+F23 "Set_reg_R5" I L 11000 10250 50
+F24 "Set_reg_R6" I L 11000 10350 50
+F25 "Set_reg_R7" I L 11000 10450 50
+F26 "Set_reg_R8" I L 11000 10550 50
+F27 "Set_reg_R9" I L 11000 10650 50
+F28 "Set_reg_R10" I L 11000 10750 50
+F29 "Set_reg_R11" I L 11000 10850 50
+F30 "Set_reg_R12" I L 11000 10950 50
+F31 "Set_reg_R13" I L 11000 11050 50
+F32 "Set_reg_R14" I L 11000 11150 50
+F33 "Set_reg_R15" I L 11000 11250 50
+F34 "Enbale_reg_R0" I L 11000 11400 50
+F35 "Enable_reg_R1" I L 11000 11500 50
+F36 "Enable_reg_R2" I L 11000 11600 50
+F37 "Enable_reg_R3" I L 11000 11700 50
+F38 "Enable_reg_R4" I L 11000 11800 50
+F39 "Enable_reg_R5" I L 11000 11900 50
+F40 "Enable_reg_R6" I L 11000 12000 50
+F41 "Enable_reg_R7" I L 11000 12100 50
+F42 "Enable_reg_R8" I L 11000 12200 50
+F43 "Enable_reg_R9" I L 11000 12300 50
+F44 "Enable_reg_R10" I L 11000 12400 50
+F45 "Enable_reg_R11" I L 11000 12500 50
+F46 "Enable_reg_R12" I L 11000 12600 50
+F47 "Enable_reg_R13" I L 11000 12700 50
+F48 "Enable_reg_R14" I L 11000 12800 50
+F49 "Enable_reg_R15" I L 11000 12900 50
+F50 "Out_bus_0" T R 12100 8100 50
+F51 "Out_bus_1" T R 12100 8200 50
+F52 "Out_bus_2" T R 12100 8300 50
+F53 "Out_bus_3" T R 12100 8400 50
+F54 "Out_bus_4" T R 12100 8500 50
+F55 "Out_bus_5" T R 12100 8600 50
+F56 "Out_bus_6" T R 12100 8700 50
+F57 "Out_bus_7" T R 12100 8800 50
+F58 "Out_bus_8" T R 12100 8900 50
+F59 "Out_bus_9" T R 12100 9000 50
+F60 "Out_bus_10" T R 12100 9100 50
+F61 "Out_bus_11" T R 12100 9200 50
+F62 "Out_bus_12" T R 12100 9300 50
+F63 "Out_bus_13" T R 12100 9400 50
+F64 "Out_bus_14" T R 12100 9500 50
+F65 "Out_bus_15" T R 12100 9600 50
 $EndSheet
+$Sheet
+S 10800 5500 1650 1700
+U 6034094B
+F0 "RAM addr control" 50
+F1 "RAM addr control.sch" 50
+F2 "Bus_0" T R 12450 5600 50
+F3 "Bus_1" T R 12450 5700 50
+F4 "Bus_2" T R 12450 5800 50
+F5 "Bus_3" T R 12450 5900 50
+F6 "Bus_4" T R 12450 6000 50
+F7 "Bus_5" T R 12450 6100 50
+F8 "Bus_6" T R 12450 6200 50
+F9 "Bus_7" T R 12450 6300 50
+F10 "Bus_8" T R 12450 6400 50
+F11 "Bus_9" T R 12450 6500 50
+F12 "Bus_10" T R 12450 6600 50
+F13 "Bus_11" T R 12450 6700 50
+F14 "Bus_12" T R 12450 6800 50
+F15 "Bus_13" T R 12450 6900 50
+F16 "Bus_14" T R 12450 7000 50
+F17 "Bus_15" T R 12450 7100 50
+F18 "Enable_internal_addr_bus_filter" I L 10800 5600 50
+F19 "Enable_instruc_addr_reg" I L 10800 5750 50
+F20 "Set_instruc_addr_reg" I L 10800 5850 50
+$EndSheet
+Text Notes 11000 13200 0    50   ~ 0
+sch =
+Text Notes 10800 7350 0    50   ~ 0
+sch =
 $EndSCHEMATC

Commit message: Update 24/02/2021
Other:
- note added: "sch = OK"

Commit message: update 28/03/2021
Connections:
- wire segments 262 -> 316
Changed lines of the file:
@@
 $Descr A2 23386 16535
 encoding utf-8
-Sheet 1 53
+Sheet 1 57
 Title ""
 Date ""
@@
 	15750 5750 15750 7650
 Wire Wire Line
-	15750 7650 13800 7650
-Wire Wire Line
-	13800 7600 15700 7600
-Wire Wire Line
 	15700 7600 15700 5650
 Wire Wire Line
 	15700 5650 15850 5650
 Wire Wire Line
-	15850 5500 15550 5500
-Wire Wire Line
-	15550 5500 15550 7500
-Wire Wire Line
-	15550 7500 13800 7500
+	15850 5500 15600 5500
+Wire Wire Line
+	15600 5500 15600 7500
 Wire Wire Line
 	15850 2750 15450 2750
@@
 	15450 2750 15450 2300
 Wire Wire Line
-	15450 2300 12800 2300
-Wire Wire Line
 	15850 2650 15500 2650
 Wire Wire Line
 	15500 2650 15500 2250
-Wire Wire Line
-	15500 2250 12800 2250
-Wire Wire Line
-	12800 2150 15650 2150
 Wire Wire Line
 	15650 2150 15650 2500
@@
 Wire Wire Line
 	18350 5500 18350 7900
+Wire Wire Line
+	17350 3200 17450 3200
+Wire Wire Line
+	17450 3200 17450 5200
+Wire Wire Line
+	17450 5200 15450 5200
+Wire Wire Line
+	15450 7450 13900 7450
+Wire Wire Line
+	13900 7450 13900 6500
+Wire Wire Line
+	13900 6500 14000 6500
+Wire Wire Line
+	15450 5200 15450 7450
+Wire Wire Line
+	17350 2900 18500 2900
+Wire Wire Line
+	17350 3000 18500 3000
+Wire Wire Line
+	17350 3100 18500 3100
+Wire Wire Line
+	17450 3200 18500 3200
+Connection ~ 17450 3200
+Wire Wire Line
+	11450 2150 15650 2150
+Wire Wire Line
+	11450 2250 15500 2250
+Wire Wire Line
+	11450 2300 15450 2300
+Wire Wire Line
+	12500 2650 11450 2650
+Wire Wire Line
+	12500 2750 11450 2750
+Wire Wire Line
+	14000 6300 11350 6300
+Wire Wire Line
+	14000 6400 11350 6400
+Wire Wire Line
+	14000 6650 11350 6650
+Wire Wire Line
+	14000 6750 11350 6750
+Wire Wire Line
+	14000 6850 11350 6850
+Wire Wire Line
+	14000 6950 11350 6950
+Wire Wire Line
+	14000 7050 11350 7050
+Wire Wire Line
+	14000 7150 11350 7150
+Wire Wire Line
+	14000 7250 11350 7250
+Wire Wire Line
+	11350 7500 15600 7500
+Wire Wire Line
+	11350 7600 15700 7600
+Wire Wire Line
+	11350 7650 15750 7650
+Wire Wire Line
+	14100 9550 11500 9550
+Wire Wire Line
+	14100 9650 11500 9650
+Wire Wire Line
+	11500 9750 14100 9750
+Wire Wire Line
+	14100 9850 11500 9850
+Wire Wire Line
+	14100 9950 11500 9950
+Wire Wire Line
+	14100 10050 11500 10050
+Wire Wire Line
+	14100 10150 11500 10150
+Wire Wire Line
+	14100 10250 11500 10250
+Wire Wire Line
+	14100 10350 11500 10350
+Wire Wire Line
+	14100 10450 11500 10450
+Wire Wire Line
+	14100 10550 11500 10550
+Wire Wire Line
+	14100 10650 11500 10650
+Wire Wire Line
+	14100 10750 11500 10750
+Wire Wire Line
+	14100 10850 11500 10850
+Wire Wire Line
+	14100 10950 11500 10950
+Wire Wire Line
+	14100 11050 11500 11050
+Wire Wire Line
+	14100 11200 11500 11200
+Wire Wire Line
+	14100 11300 11500 11300
+Wire Wire Line
+	14100 11400 11500 11400
+Wire Wire Line
+	14100 11500 11500 11500
+Wire Wire Line
+	14100 11600 11500 11600
+Wire Wire Line
+	14100 11700 11500 11700
+Wire Wire Line
+	14100 11800 11500 11800
+Wire Wire Line
+	14100 11900 11500 11900
+Wire Wire Line
+	14100 12000 11500 12000
+Wire Wire Line
+	14100 12100 11500 12100
+Wire Wire Line
+	14100 12200 11500 12200
+Wire Wire Line
+	14100 12300 11500 12300
+Wire Wire Line
+	14100 12400 11500 12400
+Wire Wire Line
+	11500 12500 14100 12500
+Wire Wire Line
+	14100 12600 11500 12600
+Wire Wire Line
+	14100 12700 11500 12700
+$Sheet
+S 6000 9550 1700 3500
+U 60CED218
+F0 "Work register decoder" 50
+F1 "Work register decoder.sch" 50
+F2 "Instruc_reg_bus_0" I L 6000 9650 50
+F3 "Instruc_reg_bus_1" I L 6000 9750 50
+F4 "Instruc_reg_bus_2" I L 6000 9850 50
+F5 "Instruc_reg_bus_3" I L 6000 9950 50
+F6 "Instruc_reg_bus_4" I L 6000 10050 50
+F7 "Instruc_reg_bus_5" I L 6000 10150 50
+F8 "Instruc_reg_bus_6" I L 6000 10250 50
+F9 "Instruc_reg_bus_7" I L 6000 10350 50
+F10 "Reg_A" I L 6000 10500 50
+F11 "Reg_B" I L 6000 10600 50
+F12 "Clock_Enable" I L 6000 10750 50
+F13 "Clock_Set" I L 6000 10850 50
+F14 "Set_reg_R0" O R 7700 9650 50
+F15 "Set_reg_R1" O R 7700 9750 50
+F16 "Set_reg_R2" O R 7700 9850 50
+F17 "Set_reg_R3" O R 7700 9950 50
+F18 "Set_reg_R4" O R 7700 10050 50
+F19 "Set_reg_R5" O R 7700 10150 50
+F20 "Set_reg_R6" O R 7700 10250 50
+F21 "Set_reg_R7" O R 7700 10350 50
+F22 "Set_reg_R8" O R 7700 10450 50
+F23 "Set_reg_R9" O R 7700 10550 50
+F24 "Set_reg_R10" O R 7700 10650 50
+F25 "Set_reg_R11" O R 7700 10750 50
+F26 "Set_reg_R12" O R 7700 10850 50
+F27 "Set_reg_R13" O R 7700 10950 50
+F28 "Set_reg_R14" O R 7700 11050 50
+F29 "Set_reg_R15" O R 7700 11150 50
+F30 "Enable_reg_R0" O R 7700 11300 50
+F31 "Enable_reg_R1" O R 7700 11400 50
+F32 "Enable_reg_R2" O R 7700 11500 50
+F33 "Enable_reg_R3" O R 7700 11600 50
+F34 "Enable_reg_R4" O R 7700 11700 50
+F35 "Enable_reg_R5" O R 7700 11800 50
+F36 "Enable_reg_R6" O R 7700 11900 50
+F37 "Enable_reg_R7" O R 7700 12000 50
+F38 "Enable_reg_R8" O R 7700 12100 50
+F39 "Enable_reg_R9" O R 7700 12200 50
+F40 "Enable_reg_R10" O R 7700 12300 50
+F41 "Enable_reg_R11" O R 7700 12400 50
+F42 "Enable_reg_R12" O R 7700 12500 50
+F43 "Enable_reg_R13" O R 7700 12600 50
+F44 "Enable_reg_R14" O R 7700 12700 50
+F45 "Enable_reg_R15" O R 7700 12800 50
+$EndSheet
+$Sheet
+S 2400 8850 1350 1950
+U 6105809C
+F0 "Instruction register" 50
+F1 "Instruction register.sch" 50
+F2 "Input_bus_0" I L 2400 8950 50
+F3 "Input_bus_1" I L 2400 9050 50
+F4 "Input_bus_2" I L 2400 9150 50
+F5 "Input_bus_3" I L 2400 9250 50
+F6 "Input_bus_4" I L 2400 9350 50
+F7 "Input_bus_5" I L 2400 9450 50
+F8 "Input_bus_6" I L 2400 9550 50
+F9 "Input_bus_7" I L 2400 9650 50
+F10 "Input_bus_8" I L 2400 9750 50
+F11 "Input_bus_9" I L 2400 9850 50
+F12 "Input_bus_10" I L 2400 9950 50
+F13 "Input_bus_11" I L 2400 10050 50
+F14 "Input_bus_12" I L 2400 10150 50
+F15 "Input_bus_13" I L 2400 10250 50
+F16 "Input_bus_14" I L 2400 10350 50
+F17 "Input_bus_15" I L 2400 10450 50
+F18 "Set_reg" I L 2400 10600 50
+F19 "Enable_reg" I L 2400 10700 50
+F20 "Output_bus_0" O R 3750 8950 50
+F21 "Output_bus_1" O R 3750 9050 50
+F22 "Output_bus_2" O R 3750 9150 50
+F23 "Output_bus_3" O R 3750 9250 50
+F24 "Output_bus_4" O R 3750 9350 50
+F25 "Output_bus_5" O R 3750 9450 50
+F26 "Output_bus_6" O R 3750 9550 50
+F27 "Output_bus_7" O R 3750 9650 50
+F28 "Output_bus_8" O R 3750 9750 50
+F29 "Output_bus_9" O R 3750 9850 50
+F30 "Output_bus_10" O R 3750 9950 50
+F31 "Output_bus_11" O R 3750 10050 50
+F32 "Output_bus_12" O R 3750 10150 50
+F33 "Output_bus_13" O R 3750 10250 50
+F34 "Output_bus_14" O R 3750 10350 50
+F35 "Output_bus_15" O R 3750 10450 50
+$EndSheet
 $EndSCHEMATC

Commit message: update
Changed lines of the file:
@@
 $EndSheet
 $Sheet
-S 2400 8850 1350 1950
+S 2400 8850 1450 1950
 U 6105809C
 F0 "Instruction register" 50
@@
 F18 "Set_reg" I L 2400 10600 50
 F19 "Enable_reg" I L 2400 10700 50
-F20 "Output_bus_0" O R 3750 8950 50
-F21 "Output_bus_1" O R 3750 9050 50
-F22 "Output_bus_2" O R 3750 9150 50
-F23 "Output_bus_3" O R 3750 9250 50
-F24 "Output_bus_4" O R 3750 9350 50
-F25 "Output_bus_5" O R 3750 9450 50
-F26 "Output_bus_6" O R 3750 9550 50
-F27 "Output_bus_7" O R 3750 9650 50
-F28 "Output_bus_8" O R 3750 9750 50
-F29 "Output_bus_9" O R 3750 9850 50
-F30 "Output_bus_10" O R 3750 9950 50
-F31 "Output_bus_11" O R 3750 10050 50
-F32 "Output_bus_12" O R 3750 10150 50
-F33 "Output_bus_13" O R 3750 10250 50
-F34 "Output_bus_14" O R 3750 10350 50
-F35 "Output_bus_15" O R 3750 10450 50
+F20 "Instruction_bus_0" O R 3850 8950 50
+F21 "Instruction_bus_1" O R 3850 9050 50
+F22 "Instruction_bus_2" O R 3850 9150 50
+F23 "Instruction_bus_3" O R 3850 9250 50
+F24 "Instruction_bus_4" O R 3850 9350 50
+F25 "Instruction_bus_5" O R 3850 9450 50
+F26 "Instruction_bus_6" O R 3850 9550 50
+F27 "Instruction_bus_7" O R 3850 9650 50
+F28 "Instruction_bus_8" O R 3850 9750 50
+F29 "Instruction_bus_9" O R 3850 9850 50
+F30 "Instruction_bus_10" O R 3850 9950 50
+F31 "Instruction_bus_11" O R 3850 10050 50
+F32 "Instruction_bus_12" O R 3850 10150 50
+F33 "Instruction_bus_13" O R 3850 10250 50
+F34 "Instruction_bus_14" O R 3850 10350 50
+F35 "Instruction_bus_15" O R 3850 10450 50
 $EndSheet
 $EndSCHEMATC

Commit message: update
Connections:
- wire segments 316 -> 317
