File: straggio computer v1.3/work registers.sch (KiCad schematic (older format))
At the start: 0 parts

Commit message: Update 22/02/2021
Other:
- note added: "full 8bit register"
- note added: "sch = OK\npcb ="
Changed lines of the file:
@@
 $Descr A1 33110 23386
 encoding utf-8
-Sheet 2 35
+Sheet 2 39
 Title "Work registers"
 Date "2021-02-21"
@@
 Wire Wire Line
 	6050 6950 6150 6950
-Text Notes 5350 8950 0    50   ~ 0
-sch = \npcb =
-Text Notes 5350 7400 0    50   ~ 0
-sch = \npcb =
 $Sheet
 S 5050 8000 1000 1150
@@
 Wire Wire Line
 	6050 10050 6150 10050
-Text Notes 5350 12050 0    50   ~ 0
-sch = \npcb =
-Text Notes 5350 10500 0    50   ~ 0
-sch = \npcb =
 $Sheet
 S 5050 11100 1000 1150
@@
 Wire Wire Line
 	9250 6950 9350 6950
-Text Notes 8550 8950 0    50   ~ 0
-sch = \npcb =
-Text Notes 8550 7400 0    50   ~ 0
-sch = \npcb =
 $Sheet
 S 8250 8000 1000 1150
@@
 Wire Wire Line
 	9250 10050 9350 10050
-Text Notes 8550 12050 0    50   ~ 0
-sch = \npcb =
-Text Notes 8550 10500 0    50   ~ 0
-sch = \npcb =
 $Sheet
 S 8250 11100 1000 1150
@@
 Wire Wire Line
 	12450 6950 12550 6950
-Text Notes 11750 8950 0    50   ~ 0
-sch = \npcb =
-Text Notes 11750 7400 0    50   ~ 0
-sch = \npcb =
 $Sheet
 S 11450 8000 1000 1150
@@
 Wire Wire Line
 	12450 10050 12550 10050
-Text Notes 11750 12050 0    50   ~ 0
-sch = \npcb =
-Text Notes 11750 10500 0    50   ~ 0
-sch = \npcb =
 $Sheet
 S 11450 11100 1000 1150
@@
 Wire Wire Line
 	15650 6950 15750 6950
-Text Notes 14950 8950 0    50   ~ 0
-sch = \npcb =
-Text Notes 14950 7400 0    50   ~ 0
-sch = \npcb =
 $Sheet
 S 14650 8000 1000 1150
@@
 Wire Wire Line
 	15650 10050 15750 10050
-Text Notes 14950 12050 0    50   ~ 0
-sch = \npcb =
-Text Notes 14950 10500 0    50   ~ 0
-sch = \npcb =
 $Sheet
 S 14650 11100 1000 1150
@@
 Wire Wire Line
 	18850 6950 18950 6950
-Text Notes 18150 8950 0    50   ~ 0
-sch = \npcb =
-Text Notes 18150 7400 0    50   ~ 0
-sch = \npcb =
 $Sheet
 S 17850 8000 1000 1150
@@
 Wire Wire Line
 	18850 10050 18950 10050
-Text Notes 18150 12050 0    50   ~ 0
-sch = \npcb =
-Text Notes 18150 10500 0    50   ~ 0
-sch = \npcb =
 $Sheet
 S 17850 11100 1000 1150
@@
 Wire Wire Line
 	22050 6950 22150 6950
-Text Notes 21350 8950 0    50   ~ 0
-sch = \npcb =
-Text Notes 21350 7400 0    50   ~ 0
-sch = \npcb =
 $Sheet
 S 21050 8000 1000 1150
@@
 Wire Wire Line
 	22050 10050 22150 10050
-Text Notes 21350 12050 0    50   ~ 0
-sch = \npcb =
-Text Notes 21350 10500 0    50   ~ 0
-sch = \npcb =
 $Sheet
 S 21050 11100 1000 1150
@@
 Wire Wire Line
 	25250 6950 25350 6950
-Text Notes 24550 8950 0    50   ~ 0
-sch = \npcb =
-Text Notes 24550 7400 0    50   ~ 0
-sch = \npcb =
 $Sheet
 S 24250 6600 1000 1150
@@
 Wire Wire Line
 	25250 10050 25350 10050
-Text Notes 24550 12050 0    50   ~ 0
-sch = \npcb =
-Text Notes 24550 10500 0    50   ~ 0
-sch = \npcb =
 $Sheet
 S 24250 11100 1000 1150
@@
 Wire Wire Line
 	28450 6950 28550 6950
-Text Notes 27750 8950 0    50   ~ 0
-sch = \npcb =
-Text Notes 27750 7400 0    50   ~ 0
-sch = \npcb =
 $Sheet
 S 27450 8000 1000 1150
@@
 F19 "Out_7" T R 28450 9050 50
 $EndSheet
-$Sheet
-S 27450 6600 1000 1150
-U 60A1314C
-F0 "R14 Low" 50
-F1 "full 8bit register.sch" 50
-F2 "Set_register" I L 27450 6700 50
-F3 "Enable_register" I L 27450 6800 50
-F4 "In_0" I L 27450 6950 50
-F5 "In_1" I L 27450 7050 50
-F6 "In_2" I L 27450 7150 50
-F7 "In_3" I L 27450 7250 50
-F8 "In_4" I L 27450 7350 50
-F9 "In_5" I L 27450 7450 50
-F10 "In_6" I L 27450 7550 50
-F11 "In_7" I L 27450 7650 50
-F12 "Out_0" T R 28450 6950 50
-F13 "Out_1" T R 28450 7050 50
-F14 "Out_2" T R 28450 7150 50
-F15 "Out_3" T R 28450 7250 50
-F16 "Out_4" T R 28450 7350 50
-F17 "Out_5" T R 28450 7450 50
-F18 "Out_6" T R 28450 7550 50
-F19 "Out_7" T R 28450 7650 50
-$EndSheet
 Wire Wire Line
 	27350 8100 26200 8100
@@
 Wire Wire Line
 	28450 10050 28550 10050
-Text Notes 27750 12050 0    50   ~ 0
-sch = \npcb =
-Text Notes 27750 10500 0    50   ~ 0
-sch = \npcb =
+Text Notes 29500 7400 0    50   ~ 0
+sch = OK\npcb =
 $Sheet
 S 27450 11100 1000 1150
@@
 F19 "Out_7" T R 25250 9050 50
 $EndSheet
+$Sheet
+S 27450 6600 1000 1150
+U 60A1314C
+F0 "R14 Low" 50
+F1 "full 8bit register.sch" 50
+F2 "Set_register" I L 27450 6700 50
+F3 "Enable_register" I L 27450 6800 50
+F4 "In_0" I L 27450 6950 50
+F5 "In_1" I L 27450 7050 50
+F6 "In_2" I L 27450 7150 50
+F7 "In_3" I L 27450 7250 50
+F8 "In_4" I L 27450 7350 50
+F9 "In_5" I L 27450 7450 50
+F10 "In_6" I L 27450 7550 50
+F11 "In_7" I L 27450 7650 50
+F12 "Out_0" T R 28450 6950 50
+F13 "Out_1" T R 28450 7050 50
+F14 "Out_2" T R 28450 7150 50
+F15 "Out_3" T R 28450 7250 50
+F16 "Out_4" T R 28450 7350 50
+F17 "Out_5" T R 28450 7450 50
+F18 "Out_6" T R 28450 7550 50
+F19 "Out_7" T R 28450 7650 50
+$EndSheet
+Text Notes 29500 7250 0    50   ~ 0
+full 8bit register
 $EndSCHEMATC
