File: straggio computer v1.3/ADDer and Subtractor (MSB).sch (KiCad schematic (older format))
At the start: 0 parts

Commit message: update
Parts:
- added C? (x2): C, symbol Device:C
- added J?: Higher byte A input, symbol Connector:Conn_01x08_Male
- added J?: Higher byte B input, symbol Connector:Conn_01x08_Male
- added J?: Control signals, symbol Connector:Conn_01x04_Male
- added J?: Higher byte output, symbol Connector:Conn_01x08_Male
- added J?: Carry output, symbol Connector:Conn_01x01_Male
- added J?: Power, symbol Connector:Conn_01x02_Male
- added Q? (x232): 2N7000, Package_TO_SOT_THT:TO-92_Inline, symbol Transistor_FET:2N7000
- added R? (x120): R, symbol Device:R
Connections:
- net A10: now also J?.3 (Pin_3), Q?.2 (G), Q?.2 (G), Q?.2 (G), Q?.3 (D)
- net A11: now also J?.4 (Pin_4), Q?.2 (G), Q?.2 (G), Q?.2 (G), Q?.3 (D)
- net A12: now also J?.5 (Pin_5), Q?.2 (G), Q?.2 (G), Q?.2 (G), Q?.3 (D)
- net A13: now also J?.6 (Pin_6), Q?.2 (G), Q?.2 (G), Q?.2 (G), Q?.3 (D)
- net A14: now also J?.7 (Pin_7), Q?.2 (G), Q?.2 (G), Q?.2 (G), Q?.3 (D)
- net A15: now also J?.8 (Pin_8), Q?.2 (G), Q?.2 (G), Q?.2 (G), Q?.3 (D)
- net A8: now also J?.1 (Pin_1), Q?.2 (G), Q?.2 (G), Q?.2 (G), Q?.3 (D)
- net A9: now also J?.2 (Pin_2), Q?.2 (G), Q?.2 (G), Q?.2 (G), Q?.3 (D)
- net B10: now also J?.3 (Pin_3), Q?.2 (G), Q?.2 (G)
- net B11: now also J?.4 (Pin_4), Q?.2 (G), Q?.2 (G)
- net B12: now also J?.5 (Pin_5), Q?.2 (G), Q?.2 (G)
- net B13: now also J?.6 (Pin_6), Q?.2 (G), Q?.2 (G)
- net B14: now also J?.7 (Pin_7), Q?.2 (G), Q?.2 (G)
- net B15: now also J?.8 (Pin_8), Q?.2 (G), Q?.2 (G)
- net B8: now also J?.1 (Pin_1), Q?.2 (G), Q?.2 (G)
- net B9: now also J?.2 (Pin_2), Q?.2 (G), Q?.2 (G)
- net C10: now also J?.6 (Pin_6), Q?.3 (D), R?.2
- net C11: now also J?.5 (Pin_5), Q?.3 (D), R?.2
- net C12: now also J?.4 (Pin_4), Q?.3 (D), R?.2
- net C13: now also J?.3 (Pin_3), Q?.3 (D), R?.2
- net C14: now also J?.2 (Pin_2), Q?.3 (D), R?.2
- net C15: now also J?.1 (Pin_1), Q?.3 (D), R?.2
- net C8: now also J?.8 (Pin_8), Q?.3 (D), R?.2
- net C9: now also J?.7 (Pin_7), Q?.3 (D), R?.2
- net Carry_out: now also J?.1 (Pin_1), Q?.3 (D), R?.2
- net Cy_in: now also J?.3 (Pin_3), Q?.2 (G), Q?.2 (G), Q?.2 (G)
- net enabler_in: now also J?.4 (Pin_4), Q?.2 (G), Q?.2 (G), Q?.2 (G), Q?.2 (G), Q?.2 (G), Q?.2 (G), Q?.2 (G), Q?.2 (G)
- net invert_in: now also J?.2 (Pin_2), Q?.2 (G), Q?.2 (G), Q?.2 (G), Q?.2 (G), Q?.2 (G), Q?.2 (G), Q?.2 (G), Q?.2 (G), Q?.2 (G), Q?.2 (G), Q?.2 (G), Q?.2 (G), Q?.2 (G), Q?.2 (G), Q?.2 (G), Q?.2 (G)
- net pull_down_in: now also J?.1 (Pin_1), Q?.2 (G), Q?.2 (G), Q?.2 (G), Q?.2 (G), Q?.2 (G), Q?.2 (G), Q?.2 (G), Q?.2 (G)
- new net: Q?.2 (G), Q?.2 (G), Q?.2 (G), Q?.3 (D), Q?.3 (D), R?.2 (x16)
- new net: Q?.2 (G), Q?.3 (D), Q?.3 (D), R?.2 (x48)
- new net: Q?.1 (S), Q?.3 (D) (x40)
- new net: Q?.2 (G), Q?.3 (D), R?.2 (x40)
- new net: Q?.2 (G), Q?.2 (G), Q?.2 (G), Q?.3 (D), R?.2 (x7)
- new net GND: C?.2, C?.2, J?.2 (Pin_2), Q?.1 (S), Q?.1 (S), Q?.1 (S), Q?.1 (S), Q?.1 (S), Q?.1 (S), Q?.1 (S), Q?.1 (S), Q?.1 (S), Q?.1 (S), Q?.1 (S), Q?.1 (S), Q?.1 (S), Q?.1 (S), Q?.1 (S), Q?.1 (S), Q?.1 (S), Q?.1 (S), Q?.1 (S), Q?.1 (S), Q?.1 (S), Q?.1 (S), Q?.1 (S), Q?.1 (S), Q?.1 (S), Q?.1 (S), Q?.1 (S), Q?.1 (S), Q?.1 (S), Q?.1 (S), Q?.1 (S), Q?.1 (S), Q?.1 (S), Q?.1 (S), Q?.1 (S), Q?.1 (S), Q?.1 (S), Q?.1 (S), Q?.1 (S), Q?.1 (S), Q?.1 (S), Q?.1 (S), Q?.1 (S), Q?.1 (S), Q?.1 (S), Q?.1 (S), Q?.1 (S), Q?.1 (S), Q?.1 (S), Q?.1 (S), Q?.1 (S), Q?.1 (S), Q?.1 (S), Q?.1 (S), Q?.1 (S), Q?.1 (S), Q?.1 (S), Q?.1 (S), Q?.1 (S), Q?.1 (S), Q?.1 (S), Q?.1 (S), Q?.1 (S), Q?.1 (S), Q?.1 (S), Q?.1 (S), Q?.1 (S), Q?.1 (S), Q?.1 (S), Q?.1 (S), Q?.1 (S), Q?.1 (S), Q?.1 (S), Q?.1 (S), Q?.1 (S), Q?.1 (S), Q?.1 (S), Q?.1 (S), Q?.1 (S), Q?.1 (S), Q?.1 (S), Q?.1 (S), Q?.1 (S), Q?.1 (S), Q?.1 (S), Q?.1 (S), Q?.1 (S), Q?.1 (S), Q?.1 (S), Q?.1 (S), Q?.1 (S), Q?.1 (S), Q?.1 (S), Q?.1 (S), Q?.1 (S), Q?.1 (S), Q?.1 (S), Q?.1 (S), Q?.1 (S), Q?.1 (S), Q?.1 (S), Q?.1 (S), Q?.1 (S), Q?.1 (S), Q?.1 (S), Q?.1 (S), Q?.1 (S), Q?.1 (S), Q?.1 (S), Q?.1 (S), Q?.1 (S), Q?.1 (S), Q?.1 (S), Q?.1 (S), Q?.1 (S), Q?.1 (S), Q?.1 (S), Q?.1 (S), Q?.1 (S), Q?.1 (S), Q?.1 (S), Q?.1 (S), Q?.1 (S), Q?.1 (S), Q?.1 (S), Q?.1 (S), Q?.1 (S), Q?.1 (S), Q?.1 (S), Q?.1 (S), Q?.1 (S), Q?.1 (S), Q?.1 (S), Q?.1 (S), Q?.1 (S), Q?.1 (S), Q?.1 (S), Q?.1 (S), Q?.1 (S), Q?.1 (S), Q?.1 (S), Q?.1 (S), Q?.1 (S), Q?.1 (S), Q?.1 (S), Q?.1 (S), Q?.1 (S), Q?.1 (S), Q?.1 (S), Q?.1 (S), Q?.1 (S), Q?.1 (S), Q?.1 (S), Q?.1 (S), Q?.1 (S), Q?.1 (S), Q?.1 (S), Q?.1 (S), Q?.1 (S), Q?.1 (S), Q?.1 (S), Q?.1 (S), Q?.1 (S), Q?.1 (S), Q?.1 (S), Q?.1 (S), Q?.1 (S), Q?.1 (S), Q?.1 (S), Q?.1 (S), Q?.1 (S), Q?.1 (S), Q?.1 (S), Q?.1 (S), Q?.1 (S), Q?.1 (S), Q?.1 (S), Q?.1 (S), Q?.1 (S), Q?.1 (S), Q?.1 (S), Q?.1 (S), Q?.1 (S), Q?.1 (S), Q?.1 (S), Q?.1 (S), Q?.1 (S), Q?.1 (S), Q?.1 (S), Q?.1 (S), Q?.1 (S), Q?.1 (S)
- new net VDD: C?.1, C?.1, J?.1 (Pin_1), R?.1, R?.1, R?.1, R?.1, R?.1, R?.1, R?.1, R?.1, R?.1, R?.1, R?.1, R?.1, R?.1, R?.1, R?.1, R?.1, R?.1, R?.1, R?.1, R?.1, R?.1, R?.1, R?.1, R?.1, R?.1, R?.1, R?.1, R?.1, R?.1, R?.1, R?.1, R?.1, R?.1, R?.1, R?.1, R?.1, R?.1, R?.1, R?.1, R?.1, R?.1, R?.1, R?.1, R?.1, R?.1, R?.1, R?.1, R?.1, R?.1, R?.1, R?.1, R?.1, R?.1, R?.1, R?.1, R?.1, R?.1, R?.1, R?.1, R?.1, R?.1, R?.1, R?.1, R?.1, R?.1, R?.1, R?.1, R?.1, R?.1, R?.1, R?.1, R?.1, R?.1, R?.1, R?.1, R?.1, R?.1, R?.1, R?.1, R?.1, R?.1, R?.1, R?.1, R?.1, R?.1, R?.1, R?.1, R?.1, R?.1, R?.1, R?.1, R?.1, R?.1, R?.1, R?.1, R?.1, R?.1, R?.1, R?.1, R?.1, R?.1, R?.1, R?.1, R?.1, R?.1, R?.1, R?.1, R?.1, R?.1, R?.1, R?.1, R?.1, R?.1, R?.1, R?.1, R?.1, R?.1, R?.1, R?.1, R?.1
Other:
- note added: "AND"
- note added: "Controlled NOTer and pull down"
- note added: "Enabler"
- note added: "Full adder"
- note added: "OR"
- note added: "XOR"
