File: straggio computer v1.3/ADDer and Subtractor.sch (KiCad schematic (older format))
At the start: 0 parts

Commit message: update
Other:
- note removed: "sch = \npcb ="
Changed lines of the file:
@@
 sch = OK\npcb =
 Text Notes 4450 6950 0    50   ~ 0
-sch = \npcb =
+sch = OK\npcb =
 $EndSCHEMATC
