File: Multiplier experiment/full multiplier 16 by 16 kikad/full multiplier 16 by 16 kikad.sch (KiCad schematic (older format))
At the start: 1408 parts

Commit message: update
Connections:
- wire segments 6659 -> 8118
