File: Experimentos/Adder and subtraction experiment/Adder and subtraction experiment.sch (KiCad schematic (older format))
At the start: 148 parts

Commit message: update
Other:
- note added: "ADDer and Subtractor (LSB)"
- note added: "ADDer and Subtractor (MSB)"
- note added: "Cy"
- note added: "Invert"
- note added: "pull down"
